Commit message: new urdf

File: src/arm_description/urdf/AR3 Main Assembly.SLDASM.urdf (robot description, URDF)
Before this commit: robot AR3 Main Assembly.SLDASM, 5 links, 4 joints
Links:
- link Link1: geometry collision mesh filename=package://AR3 Main Assembly.SLDASM/meshes/Link1.STL; visual mesh filename=package://AR3 Main Assembly.SLDASM/meshes/Link1.STL
- link Link2: geometry collision mesh filename=package://AR3 Main Assembly.SLDASM/meshes/Link2.STL; visual mesh filename=package://AR3 Main Assembly.SLDASM/meshes/Link2.STL
- link Link4: geometry collision mesh filename=package://AR3 Main Assembly.SLDASM/meshes/Link4.STL; visual mesh filename=package://AR3 Main Assembly.SLDASM/meshes/Link4.STL
- link Link_3: geometry collision mesh filename=package://AR3 Main Assembly.SLDASM/meshes/Link_3.STL; visual mesh filename=package://AR3 Main Assembly.SLDASM/meshes/Link_3.STL
- link base_link: mass 0.66695527839868 -> 0.66696; geometry collision mesh filename=package://AR3 Main Assembly.SLDASM/meshes/base_link.STL; visual mesh filename=package://AR3 Main Assembly.SLDASM/meshes/base_link.STL
Joints:
- joint J1: limit lower=0 upper=0 effort=0 velocity=0 -> (none); type revolute -> fixed
- joint J2: limit lower=0 upper=0 effort=0 velocity=0 -> (none); type revolute -> fixed
- joint J3: limit lower=0 upper=0 effort=0 velocity=0 -> (none); type revolute -> fixed
- joint J4: limit lower=0 upper=0 effort=0 velocity=0 -> (none); type revolute -> fixed

Commit message: .

File: src/arm_description/urdf/AR3 Main Assembly.SLDASM.urdf (robot description, URDF)
Before this commit: robot AR3 Main Assembly.SLDASM, 5 links, 4 joints
Links:
- link Link1: geometry collision mesh filename=package://arm_description/meshes/Link1.STL; visual mesh filename=package://arm_description/meshes/Link1.STL
- link Link2: geometry collision mesh filename=package://arm_description/meshes/Link2.STL; visual mesh filename=package://arm_description/meshes/Link2.STL
- link Link4: geometry collision mesh filename=package://arm_description/meshes/Link4.STL; visual mesh filename=package://arm_description/meshes/Link4.STL
- link Link_3: geometry collision mesh filename=package://arm_description/meshes/Link_3.STL; visual mesh filename=package://arm_description/meshes/Link_3.STL
- link base_link: geometry collision mesh filename=package://arm_description/meshes/base_link.STL; visual mesh filename=package://arm_description/meshes/base_link.STL
