Commit message: new moveit files

File: src/arm_description/urdf/arm_description.urdf (robot description, URDF)
Before this commit: robot arm_description, 5 links, 4 joints
Joints:
- joint J1: limit lower=0 upper=0 effort=0 velocity=0 -> lower=-3.141593 upper=3.141593 effort=0 velocity=0.2
- joint J2: limit lower=0 upper=0 effort=0 velocity=0 -> lower=-3.141593 upper=3.141593 effort=0 velocity=0.2
- joint J3: limit lower=0 upper=0 effort=0 velocity=0 -> lower=-3.141593 upper=3.141593 effort=0 velocity=0.2
- joint J4: limit lower=0 upper=0 effort=0 velocity=0 -> lower=-3.141593 upper=3.141593 effort=0 velocity=0.2

Commit message: .

File: src/arm_description/urdf/arm_description.urdf (robot description, URDF)
Before this commit: robot arm_description, 5 links, 4 joints
Joints:
- joint J1: limit lower=-3.141593 upper=3.141593 effort=0 velocity=0.2 -> lower=0 upper=0 effort=0 velocity=0
- joint J2: limit lower=-3.141593 upper=3.141593 effort=0 velocity=0.2 -> lower=0 upper=0 effort=0 velocity=0
- joint J3: limit lower=-3.141593 upper=3.141593 effort=0 velocity=0.2 -> lower=0 upper=0 effort=0 velocity=0
- joint J4: limit lower=-3.141593 upper=3.141593 effort=0 velocity=0.2 -> lower=0 upper=0 effort=0 velocity=0
