Commit message: updated .urdf

File: src/arm_description/urdf/arm_basis.urdf (robot description, URDF)
Before this commit: robot Arm_basis, 5 links, 4 joints
Links:
- link L1: geometry collision mesh filename=package://arm_description/meshes/L1.STL; visual mesh filename=package://arm_description/meshes/L1.STL
- link L2: geometry collision mesh filename=package://arm_description/meshes/L2.STL; visual mesh filename=package://arm_description/meshes/L2.STL
- link L3: geometry collision mesh filename=package://arm_description/meshes/L3.STL; visual mesh filename=package://arm_description/meshes/L3.STL
- link base_link: geometry collision mesh filename=package://arm_description/meshes/base_link.STL; visual mesh filename=package://arm_description/meshes/base_link.STL

Commit message: Working but not fully yet

File: src/arm_description/urdf/arm_basis.urdf (robot description, URDF)
Before this commit: robot arm_description, 6 links, 5 joints
Joints:
- removed joint fixed
- added joint virtual_joint: type fixed, parent world, child base_link, origin xyz=0 0 0
- joint J1: limit lower=-3.141593 upper=3.141593 effort=0 velocity=0.2 -> lower=-3.141593 upper=3.141593 effort=40.0 velocity=0.2; origin xyz=0 0 0.0867 rpy=3.1416 0 1.5708 -> xyz=0 0 0.0867 rpy=0 0 1.5708
- joint J2: limit lower=-3.141593 upper=3.141593 effort=0 velocity=0.2 -> lower=-3.141593 upper=3.141593 effort=40.0 velocity=0.2; origin xyz=0.064146 -0.007968 -0.083075 rpy=1.5708 0.5236 3.1416 -> xyz=0.064146 -0.007968 -0.083075 rpy=1.5708 0.5236 0
- joint J3: limit lower=-3.141593 upper=3.141593 effort=0 velocity=0.2 -> lower=-3.141593 upper=3.141593 effort=40.0 velocity=0.2
- joint J4: limit lower=-3.141593 upper=3.141593 effort=0 velocity=0.2 -> lower=-3.141593 upper=3.141593 effort=40.0 velocity=0.2

Commit message: fixed urdf andplanning_context

File: src/arm_description/urdf/arm_basis.urdf (robot description, URDF)
Before this commit: robot arm_description, 6 links, 5 joints
Joints:
- removed joint virtual_joint
- added joint fixed: type fixed, parent world, child base_link, origin xyz=0 0 0
- joint J1: origin xyz=0 0 0.0867 rpy=0 0 1.5708 -> xyz=0 0 0.0867 rpy=3.1416 0 1.5708
- joint J2: origin xyz=0.064146 -0.007968 -0.083075 rpy=1.5708 0.5236 0 -> xyz=0.064146 -0.007968 -0.083075 rpy=1.5708 0.5236 3.1416

Commit message: Revert "Working but not fully yet"
This reverts commit dd68e9890b83f597d4b184aa890c476b0653c179

File: src/arm_description/urdf/arm_basis.urdf (robot description, URDF)
Before this commit: robot arm_description, 6 links, 5 joints
Joints:
- joint J1: limit lower=-3.141593 upper=3.141593 effort=40.0 velocity=0.2 -> lower=-3.141593 upper=3.141593 effort=0 velocity=0.2
- joint J2: limit lower=-3.141593 upper=3.141593 effort=40.0 velocity=0.2 -> lower=-3.141593 upper=3.141593 effort=0 velocity=0.2
- joint J3: limit lower=-3.141593 upper=3.141593 effort=40.0 velocity=0.2 -> lower=-3.141593 upper=3.141593 effort=0 velocity=0.2
- joint J4: limit lower=-3.141593 upper=3.141593 effort=40.0 velocity=0.2 -> lower=-3.141593 upper=3.141593 effort=0 velocity=0.2

Commit message: edit effort in .urdf

File: src/arm_description/urdf/arm_basis.urdf (robot description, URDF)
Before this commit: robot arm_description, 6 links, 5 joints
Joints:
- joint J1: limit lower=-3.141593 upper=3.141593 effort=0 velocity=0.2 -> lower=-3.141593 upper=3.141593 effort=40 velocity=0.2
- joint J2: limit lower=-3.141593 upper=3.141593 effort=0 velocity=0.2 -> lower=-3.141593 upper=3.141593 effort=40 velocity=0.2
- joint J3: limit lower=-3.141593 upper=3.141593 effort=0 velocity=0.2 -> lower=-3.141593 upper=3.141593 effort=40 velocity=0.2
- joint J4: limit lower=-3.141593 upper=3.141593 effort=0 velocity=0.2 -> lower=-3.141593 upper=3.141593 effort=40 velocity=0.2

Commit message: updated model

File: src/arm_description/urdf/arm_basis.urdf (robot description, URDF)
Before this commit: robot arm_description, 6 links, 5 joints
Links:
- added link Connector, mass 0.098251; collision mesh filename=package://arm_description/meshes/Connector.STL; visual mesh filename=package://arm_description/meshes/Connector.STL
- added link EE, mass 0.10423; collision mesh filename=package://arm_description/meshes/EE.STL; visual mesh filename=package://arm_description/meshes/EE.STL
- added link Link0, mass 0.94745; collision mesh filename=package://arm_description/meshes/Link0.STL; visual mesh filename=package://arm_description/meshes/Link0.STL
- added link Link5, mass 0.12103; collision mesh filename=package://arm_description/meshes/Link5.STL; visual mesh filename=package://arm_description/meshes/Link5.STL
- link Link1: mass 0.51011 -> 0.7296
- link Link2: mass 0.53035 -> 0.64235
- link Link3: mass 0.139370701456675 -> 0.25905
- link Link4: mass 0.290695240644425 -> 0.26849
- link base_link: mass 0.66695527839868 -> 29.988
Joints:
- added joint Connector_joint: type fixed, parent EE, child Connector, origin xyz=0.050145 0 0.098 rpy=0 0 0, axis 0 0 0
- added joint J0: type fixed, parent base_link, child Link0, origin xyz=0.055058 0 0.00635 rpy=0 0 0, axis 0 0 0
- added joint J5: type revolute, parent Link4, child Link5, origin xyz=0.1873 0.034781 0 rpy=0 0 0, axis 0 -1 0, limit lower=-3.14 upper=3.14 effort=1 velocity=0.2
- added joint J6: type revolute, parent Link5, child EE, origin xyz=0.0129 -0.035781 0 rpy=0 0 0, axis 1 0 0, limit lower=-3.14 upper=3.14 effort=1 velocity=0.2
- joint J1: limit lower=-3.141593 upper=3.141593 effort=40 velocity=0.2 -> lower=-3.14 upper=3.14 effort=1 velocity=0.2; origin xyz=0 0 0.0867 rpy=3.1416 0 1.5708 -> xyz=0 0 0.0307 rpy=0 0 0; parent base_link -> Link0
- joint J2: axis 0 0 1 -> 0 1 0; limit lower=-3.141593 upper=3.141593 effort=40 velocity=0.2 -> lower=-3.14 upper=3.14 effort=1 velocity=0.2; origin xyz=0.064146 -0.007968 -0.083075 rpy=1.5708 0.5236 3.1416 -> xyz=0.064146 0.051713 0.13908 rpy=0 0 0
- joint J3: axis 0 0.01527 -0.99988 -> 0 -1 0; limit lower=-3.141593 upper=3.141593 effort=40 velocity=0.2 -> lower=-3.14 upper=3.14 effort=1 velocity=0.2; origin xyz=0.1525 -0.26414 -0.043745 rpy=3.1263 0 0.5236 -> xyz=0 -0.015 0.305 rpy=0 0 0
- joint J4: axis 0 0 -1 -> -1 0 0; limit lower=-3.141593 upper=3.141593 effort=40 velocity=0.2 -> lower=-3.14 upper=3.14 effort=1 velocity=0.2; origin xyz=-0.035639 0.00078946 -0.051694 rpy=1.5708 -1.5555 -1.5708 -> xyz=0.035639 -0.0367 0 rpy=0 0 0

File: src/arm_description/urdf/arm_description.urdf (robot description, URDF)
Before this commit: robot arm_description, 5 links, 4 joints
Links:
- added link Connector, mass 0.098251; collision mesh filename=package://arm_description/meshes/Connector.STL; visual mesh filename=package://arm_description/meshes/Connector.STL
- added link EE, mass 0.10423; collision mesh filename=package://arm_description/meshes/EE.STL; visual mesh filename=package://arm_description/meshes/EE.STL
- added link Link0, mass 0.94745; collision mesh filename=package://arm_description/meshes/Link0.STL; visual mesh filename=package://arm_description/meshes/Link0.STL
- added link Link5, mass 0.12103; collision mesh filename=package://arm_description/meshes/Link5.STL; visual mesh filename=package://arm_description/meshes/Link5.STL
- link Link1: mass 0.51011 -> 0.7296
- link Link2: mass 0.53035 -> 0.64235
- link Link3: mass 0.139370701456675 -> 0.25905
- link Link4: mass 0.290695240644425 -> 0.26849
- link base_link: mass 0.66695527839868 -> 29.988
Joints:
- added joint Connector_joint: type fixed, parent EE, child Connector, origin xyz=0.050145 0 0.098 rpy=0 0 0, axis 0 0 0
- added joint J0: type fixed, parent base_link, child Link0, origin xyz=0.055058 0 0.00635 rpy=0 0 0, axis 0 0 0
- added joint J5: type revolute, parent Link4, child Link5, origin xyz=0.1873 0.034781 0 rpy=0 0 0, axis 0 -1 0, limit lower=-3.14 upper=3.14 effort=50 velocity=0.4
- added joint J6: type revolute, parent Link5, child EE, origin xyz=0.0129 -0.035781 0 rpy=0 0 0, axis 1 0 0, limit lower=-3.14 upper=3.14 effort=50 velocity=0.4
- joint J1: limit lower=0 upper=0 effort=0 velocity=0 -> lower=-3.14 upper=3.14 effort=50 velocity=0.4; origin xyz=0 0 0.0867 rpy=3.1416 0 1.5708 -> xyz=0 0 0.0307 rpy=0 0 0; parent base_link -> Link0
- joint J2: axis 0 0 1 -> 0 1 0; limit lower=0 upper=0 effort=0 velocity=0 -> lower=-3.14 upper=3.14 effort=50 velocity=0.4; origin xyz=0.064146 -0.007968 -0.083075 rpy=1.5708 0.5236 3.1416 -> xyz=0.064146 0.051713 0.13908 rpy=0 0 0
- joint J3: axis 0 0.01527 -0.99988 -> 0 -1 0; limit lower=0 upper=0 effort=0 velocity=0 -> lower=-3.14 upper=3.14 effort=50 velocity=0.4; origin xyz=0.1525 -0.26414 -0.043745 rpy=3.1263 0 0.5236 -> xyz=0 -0.015 0.305 rpy=0 0 0
- joint J4: axis 0 0 -1 -> -1 0 0; limit lower=0 upper=0 effort=0 velocity=0 -> lower=-3.14 upper=3.14 effort=50 velocity=0.4; origin xyz=-0.035639 0.00078946 -0.051694 rpy=1.5708 -1.5555 -1.5708 -> xyz=0.035639 -0.0367 0 rpy=0 0 0
